File: bsp.sch (KiCad schematic (older format))
At the start: 20 parts

Commit message: Added Gerbers
Parts:
- added C13, C14: 0.1uF, Capacitor_SMD:C_0805_2012Metric, symbol Device:C_Small
- added R3, R4, R5: 10K, Resistor_SMD:R_0805_2012Metric, symbol Device:R_Small
- added SW1, SW2: SW_Push, random-keyboard-parts:SKQG-1155865, symbol Switch:SW_Push
- C1, C11, C12, C5, C6, C7, C8: renamed from C?; footprint Capacitor_SMD:C_0603_1608Metric -> Capacitor_SMD:C_0805_2012Metric; symbol Device:C -> Device:C_Small
- C10, C9: renamed from C?; value 8pF -> 10pF; footprint Capacitor_SMD:C_0603_1608Metric -> Capacitor_SMD:C_0805_2012Metric; symbol Device:C -> Device:C_Small
- C2: renamed from C?; value 0.1uF -> 10nF; footprint Capacitor_SMD:C_0603_1608Metric -> Capacitor_SMD:C_0805_2012Metric; symbol Device:C -> Device:C_Small
- C3, C4: renamed from C?; value 1.5pF -> 12.5pF; footprint Capacitor_SMD:C_0603_1608Metric -> Capacitor_SMD:C_0805_2012Metric; symbol Device:C -> Device:C_Small
- F1: renamed from F?; footprint Resistor_SMD:R_0805_2012Metric -> Fuse:Fuse_1206_3216Metric; symbol Device:Polyfuse -> Device:Polyfuse_Small
- L1: renamed from L?; value 1.6uH -> WE-CBF Ferrite Bead; symbol Device:L -> Device:Ferrite_Bead_Small
- R1, R2: renamed from R?; footprint Resistor_SMD:R_0603_1608Metric -> Resistor_SMD:R_0805_2012Metric; symbol Device:R -> Device:R_Small
- Y1, Y2: renamed from Y?; footprint Crystal:Crystal_SMD_0603-2Pin_6.0x3.5mm -> Crystal:Crystal_SMD_3225-4Pin_3.2x2.5mm; symbol Device:Crystal -> Device:Crystal_GND24_Small
- gave numbers to parts that had none: 2
Connections:
- net +3V3: now also R3.2, SW2.2
- net GND: now also Y1.2, Y1.4, Y2.2, Y2.4, C13.1, C14.2, R4.2, R5.1, SW1.2
- net OSC32_OUT: now also Y1.3; no longer Y1.2
- net OSC_OUT: now also Y2.3; no longer Y2.2
- new net BOOT0: C14.1, R4.1, SW2.1
- new net BOOT1: R5.2
- new net NRST: C13.2, R3.1, SW1.1
Other:
- note added: "Crystal Oscillators"
- note added: "Noise Filtering"
- note added: "Power Supply"
- note added: "Reset and DFU"
- note added: "USB3"
- moved on the sheet: C1, C10, C11, C12, C2, C3, C4, C5, C6, C7, C8, C9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
