File: dirac_delta.kicad_pcb (KiCad board)
At the start: 2 copper layers, 243.2 x 76.2 mm, 0 parts

Commit message: Added Gerbers
Parts:
- added C1: 1uF, Capacitor_SMD:C_0805_2012Metric, B.Cu at (73.0, 34.1)
- added C10: 10pF, Capacitor_SMD:C_0805_2012Metric, B.Cu at (66.7, 41.3)
- added C11: 0.1uF, Capacitor_SMD:C_0805_2012Metric, B.Cu at (92.1, 30.2)
- added C12: 0.1uF, Capacitor_SMD:C_0805_2012Metric, B.Cu at (92.1, 38.1)
- added C13: 0.1uF, Capacitor_SMD:C_0805_2012Metric, B.Cu at (67.9, 54.0)
- added C14: 0.1uF, Capacitor_SMD:C_0805_2012Metric, B.Cu at (82.5, 54.0)
- added C2: 10nF, Capacitor_SMD:C_0805_2012Metric, B.Cu at (70.6, 34.1)
- added C3: 12.5pF, Capacitor_SMD:C_0805_2012Metric, B.Cu at (66.7, 38.9)
- added C4: 12.5pF, Capacitor_SMD:C_0805_2012Metric, B.Cu at (66.7, 36.5)
- added C5: 0.1uF, Capacitor_SMD:C_0805_2012Metric, B.Cu at (82.5, 34.1)
- added C6: 0.1uF, Capacitor_SMD:C_0805_2012Metric, B.Cu at (73.0, 48.4)
- added C7: 0.1uF, Capacitor_SMD:C_0805_2012Metric, B.Cu at (82.5, 48.4)
- added C8: 0.1uF, Capacitor_SMD:C_0805_2012Metric, B.Cu at (76.2, 48.4)
- added C9: 10pF, Capacitor_SMD:C_0805_2012Metric, B.Cu at (66.7, 43.7)
- added D1: D_Small, Diode_SMD:D_SOD-123, B.Cu at (41.3, 34.1)
- added D2: D_Small, Diode_SMD:D_SOD-123, B.Cu at (41.3, 53.2)
- added D3: D_Small, Diode_SMD:D_SOD-123, B.Cu at (60.3, 34.1)
- added D4: D_Small, Diode_SMD:D_SOD-123, B.Cu at (60.3, 53.2)
- added F1: 500mA, Fuse:Fuse_1206_3216Metric, B.Cu at (82.7, 28.8)
- added L1: WE-CBF Ferrite Bead, Inductor_SMD:L_0805_2012Metric, B.Cu at (77.0, 34.9)
- added MX1: MX-NoLED, MX_Only:MXOnly-1U-Hotswap, F.Cu at (33.3, 32.5)
- added MX2: MX-NoLED, MX_Only:MXOnly-1U-Hotswap, F.Cu at (33.3, 51.6)
- added MX3: MX-NoLED, MX_Only:MXOnly-1U-Hotswap, F.Cu at (52.4, 32.5)
- added MX4: MX-NoLED, MX_Only:MXOnly-1U-Hotswap, F.Cu at (52.4, 51.6)
- added R1: 5.1K, Resistor_SMD:R_0805_2012Metric, B.Cu at (76.2, 29.4)
- added R2: 5.1K, Resistor_SMD:R_0805_2012Metric, B.Cu at (78.6, 29.4)
- added R3: 10K, Resistor_SMD:R_0805_2012Metric, B.Cu at (72.2, 54.0)
- added R4: 10K, Resistor_SMD:R_0805_2012Metric, B.Cu at (79.4, 54.0)
- added R5: 10K, Resistor_SMD:R_0805_2012Metric, B.Cu at (80.2, 34.1)
- added SW1: SW_Push, random-keyboard-parts:SKQG-1155865, B.Cu at (70.6, 59.5)
- added SW2: SW_Push, random-keyboard-parts:SKQG-1155865, B.Cu at (81.0, 59.5)
- added U1: STM32F411CEUx, Package_DFN_QFN:QFN-48-1EP_7x7mm_P0.5mm_EP5.6x5.6mm, B.Cu at (79.4, 41.3)
- added U2: TLV70233_SOT23-5, Package_TO_SOT_SMD:SOT-23-5, B.Cu at (92.1, 34.1)
- added USB1: HRO-TYPE-C-31-M-12, Type-C:HRO-TYPE-C-31-M-12, B.Cu at (74.6, 17.5)
- added Y1: 32.768KHZ, Crystal:Crystal_SMD_3225-4Pin_3.2x2.5mm, B.Cu at (70.4, 38.5)
- added Y2: 25MHZ, Crystal:Crystal_SMD_3225-4Pin_3.2x2.5mm, B.Cu at (70.4, 43.2)
Routing:
- net GND: track 0.00 -> 148.8 mm, vias 0 -> 2
- net COL0: track 0.00 -> 118.7 mm, vias 0 -> 2
- net VDD: track 0.00 -> 91.3 mm, vias 0 -> 6
- net COL1: track 0.00 -> 91.1 mm, vias 0 -> 4
- net ROW1: track 0.00 -> 44.8 mm, vias 0 -> 2
- net USB_DP: track 0.00 -> 36.9 mm, vias 0 -> 2
- net ROW0: track 0.00 -> 36.0 mm, vias 0 -> 2
- net USB_DN: track 0.00 -> 35.9 mm, vias 0 -> 2
- net NRST: track 0.00 -> 27.3 mm, vias 0 -> 2
- net BOOT0: track 0.00 -> 20.4 mm, vias 0 -> 2
- net +5V: track 0.00 -> 18.5 mm
- net Net-(F1-Pad2): track 0.00 -> 14.4 mm
- net OSC_OUT: track 0.00 -> 13.5 mm
- net VDDA: track 0.00 -> 12.3 mm
- net OSC32_IN: track 0.00 -> 11.9 mm
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- added copper zone on B.Cu, net GND
Other:
- board size 243.2 x 76.2 mm -> 74.6 x 45.2 mm
- net class Default: clearance 0.2 -> 0.1524; trace_width 0.25 -> 0.254
- rule trace_clearance: 0.2 -> 0.1524
