File: dirac_delta.sch (KiCad schematic (older format))
At the start: 5 parts, among them U1 STM32F411CEUx

Commit message: Added BSP
Parts:
- removed F1: 500mA, Resistor_SMD:R_0805_2012Metric, symbol Device:Polyfuse
- removed R1, R2: 5.1K, Resistor_SMD:R_0603_1608Metric, symbol Device:R
- removed USB1: HRO-TYPE-C-31-M-12, Type-C:HRO-TYPE-C-31-M-12, symbol Type-C:HRO-TYPE-C-31-M-12
Connections:
- net crystals/OSC32_IN: no longer names the net of U1.3 (PC14)
- net crystals/OSC32_OUT: no longer names the net of U1.4 (PC15)
- net crystals/OSC_IN: no longer names the net of U1.5 (PH0)
- net crystals/OSC_OUT: no longer names the net of U1.6 (PH1)
- no-connect marks 4 -> 2
Other:
- moved on the sheet: U1

Commit message: Added Gerbers
Connections:
- net OSC32_IN: now reaches U1.3 (PC14)
- net OSC32_OUT: now reaches U1.4 (PC15)
- net OSC_IN: now reaches U1.5 (PH0)
- net OSC_OUT: now reaches U1.6 (PH1)
- net PA0 renamed ROW1
- net PA1 renamed ROW0
- net PA10 renamed COL1
- net PA13: no longer names the net of U1.34 (PA13)
- net PA14: no longer names the net of U1.37 (PA14)
- net PA15: no longer names the net of U1.38 (PA15)
- net PA2: no longer names the net of U1.12 (PA2)
- net PA3: no longer names the net of U1.13 (PA3)
- net PA4: no longer names the net of U1.14 (PA4)
- net PA5: no longer names the net of U1.15 (PA5)
- net PA6: no longer names the net of U1.16 (PA6)
- net PA7: no longer names the net of U1.17 (PA7)
- net PA8: no longer names the net of U1.29 (PA8)
- net PA9 renamed COL0
- net PB0: no longer names the net of U1.18 (PB0)
- net PB1: no longer names the net of U1.19 (PB1)
- net PB10: no longer names the net of U1.21 (PB10)
- net PB12: no longer names the net of U1.25 (PB12)
- net PB13: no longer names the net of U1.26 (PB13)
- net PB14: no longer names the net of U1.27 (PB14)
- net PB15: no longer names the net of U1.28 (PB15)
- net PB2 renamed BOOT1
- net PB3: no longer names the net of U1.39 (PB3)
- net PB4: no longer names the net of U1.40 (PB4)
- net PB5: no longer names the net of U1.41 (PB5)
- net PB6: no longer names the net of U1.42 (PB6)
- net PB7: no longer names the net of U1.43 (PB7)
- net PB8: no longer names the net of U1.45 (PB8)
- net PB9: no longer names the net of U1.46 (PB9)
- no-connect marks 2 -> 26
Other:
- moved on the sheet: U1
